File: Hardware/_autosave-ESC_Hardware.sch (KiCad schematic (older format))
At the start: 24 parts

Commit message: finished schematic
Parts:
- added Conn5: ABS_ENC, symbol MRDT_Connectors:Molex_SL_03
- gave numbers to parts that had none: 21
Connections:
- net +3V3: now also Conn5.1
- net GND: now also Conn5.2
- new net Microcontroller/ABS_PWM: Conn5.3
Other:
- moved on the sheet: C2, R1, R6
